File: RFBackscatterV1/RFBackscatterV1.kicad_pcb (KiCad board)
At the start: 2 copper layers, 19.3 x 42.2 mm, 12 parts, among them J1 SMA-J-P-H-RA-TH1, U1 SIT1534AI-H4-DCC-00.001E, U3 74LVC1GU04DRL

Commit message: alexandre's advice pt2
Parts:
- added C1: 10nF, Capacitor_SMD:C_0402_1005Metric, F.Cu at (161.5, 80.8)
- added C5: 10nF, Capacitor_SMD:C_0402_1005Metric, F.Cu at (167.0, 80.8)
- BT1: footprint WADARfootprints:BAT-SMD_MY-LR44-02 -> Battery:BatteryHolder_Keystone_1060_1x2032
- C3: value 100pF -> 10nF; footprint JLab_FP:CAPC10555_55N_KEM -> Capacitor_SMD:C_0402_1005Metric
- moved TP6 14.3 mm to (150.0, 76.5)
- moved TP1 14.3 mm to (150.0, 73.2)
- moved C4 13.2 mm to (160.3, 73.8), turned to 180 degrees
- moved BT1 9.72 mm to (163.9, 56.8)
- moved C3 9.17 mm to (164.0, 86.2), turned to -90 degrees
- moved U3 7.77 mm to (164.8, 74.2), turned to 180 degrees
- moved J1 6.38 mm to (163.8, 93.2)
- moved C2 5.28 mm to (170.0, 82.2), turned to 180 degrees
- moved U2 3.81 mm to (168.8, 82.2), turned to -90 degrees
- moved U1 3.26 mm to (169.8, 74.8), turned to 90 degrees
- moved TP5 1.06 mm to (179.2, 87.5)
- moved TP3 0.75 mm to (179.2, 83.5)
Connections:
- net +1V8 renamed 3V0
- U2 pad 1: GND -> Net-(U2-OUTPUT1)
- U2 pad 3: GND -> Net-(U2-OUTPUT2)
Routing:
- net 3V0: track 30.3 -> 37.9 mm
- net Net-(C3-Pad2): track 10.6 -> 6.76 mm
- net Net-(U2-OUTPUT1): track 0.00 -> 2.83 mm
- net Net-(U2-OUTPUT2): track 0.00 -> 2.47 mm
- net GND: track 14.6 -> 12.3 mm, vias 8 -> 10
- net Net-(U2-INPUT): track 1.79 -> 3.03 mm
- net Net-(U2-VCTL2): track 19.0 -> 18.1 mm, vias 2 -> 0
- net Net-(U1-CLK_Out): track 30.1 -> 29.6 mm, vias 2 -> 0
Other:
- board size 19.3 x 42.2 mm -> 34.6 x 51.9 mm
- board text added: "RF-Backscatter-V2.0 J-Lab UCSC"
- board text removed: "RF-Backscatter-V2.0 J-Lab UCSC ericdvet jlin"

Commit message: pre-board review
Parts:
- C2, C4: footprint WADARfootprints:CAPC10555_55N_KEM -> Capacitor_SMD:C_0402_1005Metric
Routing:
- net GND: vias 10 -> 34
