File: RFBackscatterV1/RFBackscatterV1.kicad_sch (KiCad schematic)
At the start: 15 parts, among them J1 SMA-J-P-H-RA-TH1, U1 SIT1534AI-H4-DCC-00.001E, U3 74LVC1GU04DRL

Commit message: pre board review 2
Parts:
- C3, C5: footprint Capacitor_SMD:C_0402_1005Metric -> Capacitor_SMD:C_0805_2012Metric
Changed lines of the file:
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@@
 			)
 		)
-		(property "Footprint" "Capacitor_SMD:C_0402_1005Metric"
+		(property "Footprint" "Capacitor_SMD:C_0805_2012Metric"
 			(at 163.83 102.87 0)
 			(effects
@@
 			)
 		)
-		(property "Footprint" "Capacitor_SMD:C_0402_1005Metric"
+		(property "Footprint" "Capacitor_SMD:C_0805_2012Metric"
 			(at 180.34 80.01 0)
 			(effects
@@
 			)
 		)
-		(property "Datasheet" "CC0402KRX7R6BB103"
+		(property "Datasheet" ""
 			(at 180.34 80.01 0)
 			(effects

Commit message: JLPCB order
Parts:
- removed C1: 10nF, Capacitor_SMD:C_0402_1005Metric, symbol CBR04C101J3GAC:CBR04C101J3GAC
- removed C5: 10nF, Capacitor_SMD:C_0805_2012Metric, symbol CBR04C101J3GAC:CBR04C101J3GAC
- removed R1: DNP, symbol Device:R
- removed TP3: CLK_OUT, JLab_FP:EpicTestPointV1, symbol Connector:TestPoint
- removed TP6: GND, JLab_FP:EpicTestPointV1, symbol Connector:TestPoint
- removed U3: 74LVC1GU04DRL, Package_TO_SOT_SMD:SOT-553, symbol 74xGxx:74LVC1GU04DRL
- added C1: 33pF, Capacitor_SMD:C_0402_1005Metric, symbol GJM1555C1H330JB01D:GJM1555C1H330JB01D
- C3: value 10nF -> 100pF
- C4: value 33pF -> 100pF
Connections:
- net 3V0 is gone; now on an unnamed net: BT1.1 (+), TP1.1, U1.4 (Vdd)
- net GND: now also C1.2
- net at U2.4 (VCTL2): now also C1.1; no longer C4.1
- net at U2.1 (OUTPUT1): now also C3.1
- net at U2.5 (INPUT): now also C4.1; no longer C3.1
- no-connect marks 1 -> 2
Other:
- moved on the sheet: BT1, C2, C3, J1, TP1, U2
